File: avr_hardware/kicad/avrcraft-poe.sch (KiCad schematic (older format))
At the start: 60 parts, among them J1 AVRISP6, P1 ETHERNET, P2 CONN_1, P3 CONN_1, P4 CONN_1, P5 CONN_1, P6 CONN_1, P7 CONN_1, P8 CONN_1, Q1 MOSFET_P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

Commit message: update all the boards ! yay.
Changed lines of the file:
@@
-EESchema Schematic File Version 2  date Sun 03 Feb 2013 07:08:31 PM EST
+EESchema Schematic File Version 2  date Sat 09 Feb 2013 02:58:00 PM EST
 LIBS:power
 LIBS:device
@@
 LIBS:mcp1824_ct
 LIBS:zener-sot23-3
+LIBS:avrcraft-poe-cache
 EELAYER 25  0
 EELAYER END
@@
 Sheet 1 1
 Title ""
-Date "3 feb 2013"
+Date "9 feb 2013"
 Rev ""
 Comp ""
@@
 Comment4 ""
 $EndDescr
+Wire Wire Line
+	1700 3200 1700 2600
+Connection ~ 1700 2700
+Wire Wire Line
+	2000 2700 1700 2700
 Wire Wire Line
 	9650 4400 9800 4400
@@
 	4050 1300 4050 1350
 Connection ~ 1700 3200
-Wire Wire Line
-	2000 2700 1700 2700
-Wire Wire Line
-	1700 2700 1700 3200
 Connection ~ 6200 6350
 Wire Wire Line

Commit message: switch up versions to 1.5.2
Parts:
- added P10: SCL, .1SMTPIN, symbol CONN_1
- added P9: SDA, .1SMTPIN, symbol CONN_1
- added R17, R18: 4k7, SM0603, symbol R
Connections:
- net +3.3V: now also R17.1, R18.1
- net at U1.10 ((PCINT22/OC0A/AIN0)PD6): now also P9.1, R17.2
- net at U1.9 ((PCINT21/OC0B/T1)PD5): now also P10.1, R18.2
Other:
- note added: "OPTIONAL FOR I2C"

Commit message: stuff changed.
Parts:
- C15: Field4 (none) -> PCE5024CT-ND
- D5: Field4 (none) -> MBRX120LF-TPMSCT-ND
- D6: Field4 (none) -> BZX84C20LT1G
- D7: Field4 (none) -> 3SMAJ5919B-TP
- Q1: value MOSFET_P -> SQ2361EES-T1-GE3CT-ND
- U2: value MCP1824 -> MCP1824v3.3
Changed lines of the file:
@@
-EESchema Schematic File Version 2  date Wed 03 Jul 2013 03:02:33 PM EDT
+EESchema Schematic File Version 2  date Thu 01 Aug 2013 01:37:52 AM EDT
 LIBS:power
 LIBS:device
@@
 Sheet 1 1
 Title ""
-Date "3 jul 2013"
+Date "1 aug 2013"
 Rev ""
 Comp ""
@@
 F 1 "ZENER-5.6V/2W" H 10500 6550 40  0000 C CNN
 F 2 "DO214" H 10500 6400 60  0000 C CNN
+F 4 "3SMAJ5919B-TP" H 10500 6650 60  0000 C CNN "Field4"
 	1    10500 6650
 	1    0    0    -1
@@
 F 1 "ZENER-20V" H 9900 6700 40  0000 C CNN
 F 2 "SOT23EBC" H 9900 6800 60  0000 C CNN
+F 4 "BZX84C20LT1G" H 9900 6950 60  0000 C CNN "Field4"
 	1    9900 6800
 	0    1    1    0
@@
 F 0 "C15" H 8000 6350 50  0000 L CNN
 F 1 "100u" H 8000 6150 50  0000 L CNN
-F 2 "PanasonicD8Cap" H 7950 6250 60  0000 C CNN
+F 2 "PanasonicD8Cap" H 7950 6400 60  0000 C CNN
+F 4 "PCE5024CT-ND" H 7950 6000 60  0000 C CNN "Field4"
 	1    7950 6250
 	1    0    0    -1
@@
 P 8650 6750
 F 0 "Q1" H 8650 6940 60  0000 R CNN
-F 1 "MOSFET_P" H 8650 6570 60  0000 R CNN
+F 1 "SQ2361EES-T1-GE3CT-ND" H 8800 6350 60  0000 R CNN
 F 2 "SOT23GDS" H 8650 6750 60  0000 C CNN
 	1    8650 6750
@@
 F 1 "DIODESCH" H 7400 6100 40  0000 C CNN
 F 2 "SM1005" H 7400 6200 60  0001 C CNN
+F 4 "MBRX120LF-TPMSCT-ND" H 7400 6200 60  0000 C CNN "Field4"
 	1    7400 6200
 	-1   0    0    1
@@
 P 4650 5050
 F 0 "U2" H 4400 5350 60  0000 C CNN
-F 1 "MCP1824" H 4750 4750 60  0000 C CNN
+F 1 "MCP1824v3.3" H 4750 4750 60  0000 C CNN
 F 2 "SOT23-5" H 4650 5050 60  0001 C CNN
 	1    4650 5050
