File: avr_hardware/kicad/avrcraft-poeb.sch (KiCad schematic (older format))
At the start: 61 parts, among them J1 AVRISP6, J2 AVRISP6, P1 ETHERNET, P4 CONN_1, P5 CONN_1, P6 CONN_1, P7 CONN_1, P8 CONN_1, Q1 SQ2361EES-T1-GE3CT-ND, T1 S553-5999-52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

Commit message: updated hardware
Parts:
- C12: footprint SM0805 -> SM0603
- D5: footprint SM1005 -> DO214; Field4 MBRX120LF-TPMSCT-ND -> (none); NEW PART (none) -> B360A-FDICT-ND; OLD PART (none) -> MBRX120LF-TPMSCT-ND
- P4: value CONN_1 -> GND
- P5: value CONN_1 -> PD34
- P6: value CONN_1 -> 5V
- P7: value CONN_1 -> 3V3
- P8: value CONN_1 -> PB0
Changed lines of the file:
@@
-EESchema Schematic File Version 2  date Fri 09 Aug 2013 04:15:58 PM EDT
+EESchema Schematic File Version 2  date Mon 12 Aug 2013 06:35:09 PM EDT
 LIBS:power
 LIBS:device
@@
 LIBS:opa832
 LIBS:zener-sot23-3
+LIBS:avrcraft-poeb-cache
 EELAYER 25  0
 EELAYER END
@@
 Sheet 1 1
 Title ""
-Date "9 aug 2013"
+Date "12 aug 2013"
 Rev ""
 Comp ""
@@
 P 1550 2650
 F 0 "P8" H 1630 2650 40  0000 L CNN
-F 1 "CONN_1" H 1550 2705 30  0001 C CNN
+F 1 "PB0" H 1550 2705 30  0001 C CNN
 F 2 ".1SMTPIN" H 1550 2650 60  0000 C CNN
 	1    1550 2650
@@
 P 5400 1000
 F 0 "P6" H 5480 1000 40  0000 L CNN
-F 1 "CONN_1" H 5400 1055 30  0001 C CNN
+F 1 "5V" H 5400 1055 30  0001 C CNN
 F 2 ".1SMTPIN" H 5400 1000 60  0000 C CNN
 	1    5400 1000
@@
 P 6550 1250
 F 0 "P7" H 6630 1250 40  0000 L CNN
-F 1 "CONN_1" H 6550 1305 30  0001 C CNN
+F 1 "3V3" H 6550 1305 30  0001 C CNN
 F 2 ".1SMTPIN" H 6550 1250 60  0000 C CNN
 	1    6550 1250
@@
 P 4200 1550
 F 0 "P5" H 4280 1550 40  0000 L CNN
-F 1 "CONN_1" H 4200 1605 30  0001 C CNN
+F 1 "PD34" H 4200 1605 30  0001 C CNN
 F 2 ".1SMTPIN" H 4200 1550 60  0000 C CNN
 	1    4200 1550
@@
 P 5400 1250
 F 0 "P4" H 5480 1250 40  0000 L CNN
-F 1 "CONN_1" H 5400 1305 30  0001 C CNN
+F 1 "GND" H 5400 1305 30  0001 C CNN
 F 2 ".1SMTPIN" H 5400 1250 60  0000 C CNN
 	1    5400 1250
@@
 F 0 "D5" H 7400 6300 40  0000 C CNN
 F 1 "DIODESCH" H 7400 6100 40  0000 C CNN
-F 2 "SM1005" H 7400 6200 60  0001 C CNN
-F 4 "MBRX120LF-TPMSCT-ND" H 7400 6200 60  0000 C CNN "Field4"
+F 2 "DO214" H 7400 6200 60  0001 C CNN
+F 4 "MBRX120LF-TPMSCT-ND" H 7400 6200 60  0001 C CNN "OLD PART"
+F 5 "B360A-FDICT-ND" H 7400 6200 60  0000 C CNN "NEW PART"
 	1    7400 6200
 	-1   0    0    1
@@
 F 0 "C12" H 8300 6350 50  0000 L CNN
 F 1 ".22u" H 8300 6150 50  0000 L CNN
-F 2 "SM0805" H 8250 6250 60  0001 C CNN
+F 2 "SM0603" H 8250 6250 60  0001 C CNN
 	1    8250 6250
 	1    0    0    -1
