File: avr_hardware/kicad/avrcraft-poec.sch (KiCad schematic (older format))
At the start: 63 parts, among them J1 AVRISP6, J2 AVRISP6, P1 ETHERNET, P10 GND, P2 ADC0, P3 ADC1, P4 GND, P5 PD34, P6 5V, P7 3V3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

Commit message: update poc
Parts:
- added P11: +5V, 1PIN_SMD, symbol CONN_1
- added P12, P13: GND, 1PIN_SMD, symbol CONN_1
- added P14: +3.3V, 1PIN_SMD, symbol CONN_1
- added P15: POE+, 1PIN_SMD, symbol CONN_1
- C13: value 0.01u -> .01u
- R1, R2: value 680 -> 1k
- R14: value 4.7k -> 4k7
- X1: value XTAL4P -> 20MHz
Connections:
- wire segments 327 -> 333

Commit message: update POEC
Parts:
- added R16: 22k, SM0805, symbol R
- R15: footprint SM0603 -> SM0805

Commit message: fix values
Parts:
- R11, R9: value 22k -> 25k
- R15: value 22k -> 220k
- R16: value 22k -> NC
Changed lines of the file:
@@
 P 9450 6500
 F 0 "R15" V 9550 6600 50  0000 C CNN
-F 1 "22k" V 9450 6500 50  0000 C CNN
+F 1 "220k" V 9450 6500 50  0000 C CNN
 F 2 "SM0805" V 9350 6450 60  0000 C CNN
 F 3 "" H 9450 6500 60  0001 C CNN
@@
 P 10600 5850
 F 0 "R11" V 10680 5850 50  0000 C CNN
-F 1 "22k" V 10600 5850 50  0000 C CNN
+F 1 "25k" V 10600 5850 50  0000 C CNN
 F 2 "SM0603" H 10600 5850 60  0000 C CNN
 F 3 "" H 10600 5850 60  0001 C CNN
@@
 P 10550 5050
 F 0 "R9" V 10630 5050 50  0000 C CNN
-F 1 "22k" V 10550 5050 50  0000 C CNN
+F 1 "25k" V 10550 5050 50  0000 C CNN
 F 2 "SM0603" H 10550 5050 60  0000 C CNN
 F 3 "" H 10550 5050 60  0001 C CNN
@@
 P 8850 6350
 F 0 "R16" V 8950 6450 50  0000 C CNN
-F 1 "22k" V 8850 6350 50  0000 C CNN
+F 1 "NC" V 8850 6350 50  0000 C CNN
 F 2 "SM0805" V 8750 6300 60  0000 C CNN
 F 3 "" H 8850 6350 60  0001 C CNN

Commit message: update:  fix the IP stack to be able to handle "lease time" only DHCP packets. Also, update a variable in the schematico
Parts:
- R15: value 220k -> 270k
Changed lines of the file:
@@
 P 9450 6500
 F 0 "R15" V 9550 6600 50  0000 C CNN
-F 1 "220k" V 9450 6500 50  0000 C CNN
+F 1 "270k" V 9450 6500 50  0000 C CNN
 F 2 "SM0805" V 9350 6450 60  0000 C CNN
 F 3 "" H 9450 6500 60  0001 C CNN
