File: avr_hardware/kicad/avrcraft-m644.sch (KiCad schematic (older format))
At the start: 49 parts, among them IC1 ATMEGA1284P-A, J1 AVRISP6, P1 ETHERNET, P10 PWR, P11 +5V, P12 GND, P13 GND, P14 PWR, P15 GND, P16 GND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

Commit message: Update for use with dedicated serial port.
Connections:
- net labels added: SCL, SDA
