File: avr_hardware/kicad/avrcraft-poed.sch (KiCad schematic (older format))
At the start: 54 parts, among them CN1 10p, CN2 .1u, CN3 10p, CN4 10n, J1 AVRISP6, P1 ETHERNET, P10 GND, P11 +5V, P12 GND, P13 GND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

Commit message: update POED for manufacture
Parts:
- removed CN2: .1u, NETWORK1206, symbol 1206NETWORK
- added CN2, CN5: .1u, NETWORK0606, symbol NETWORK0606
- added H1, H2, H3, H4: ?, 632HOLE, symbol CONN_1
- C1: value .22u -> NP
Connections:
- net labels added: PB0/CLKO, PB1/OC1A, PD2/INT0, PD3/INT1/OC2B, PD5/OC0B, SCL/PC5/PD6/OC0A, SDA/PC4/PD7

Commit message: Update for use with dedicated serial port.
Connections:
- net labels added: MISO, MOSI, RST, SCK
Changed lines of the file:
@@
 LIBS:bridge-MB2S-TP
 LIBS:ap1117
+LIBS:avrcraft-poed-cache
 EELAYER 27 0
 EELAYER END
@@
 Sheet 1 1
 Title ""
-Date "19 jul 2014"
+Date "28 jul 2014"
 Rev ""
 Comp ""
@@
 Text Label 1150 2500 0    60   ~ 0
 PD5/OC0B
+Text Label 1350 3200 0    60   ~ 0
+MOSI
+Text Label 1600 3350 0    60   ~ 0
+MISO
+Text Label 1600 3800 0    60   ~ 0
+SCK
+Text Label 1600 3900 0    60   ~ 0
+RST
 $EndSCHEMATC

Commit message: changes - update with new design for LED
Parts:
- removed P16: ADC2, .1SMTPIN, symbol CONN_1
Connections:
- net labels added: BLUE, SCL/PC5/PD7, SDA/PC4/OC0A
- net labels removed: SCL/PC5/PD6/OC0A, SDA/PC4/PD7
- wire segments 409 -> 411
