File: usb_minecraft/hw/usb_minecraft.kicad_pcb (KiCad board)
At the start: 2 copper layers, 12 x 16.5 mm, 9 parts, among them J1 AVRISP6, P1 USB, U1 ATMEGAXU2, U2 10p, U3 1u, U4 33, X1 16MHz

Commit message: Yay updates
Other:
- board text added: "NOTE: Can shorten the USB part a tad. I.e. 1/6th the length of the item."
Changed lines of the file:
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@@
     (area 47.23663 37.760067 68.005845 56.6096)
     (thickness 1.6)
-    (drawings 31)
+    (drawings 32)
     (tracks 324)
     (zones 0)
@@
     (mod_text_size 1 1)
     (mod_text_width 0.15)
-    (pad_size 1.016 2.54)
+    (pad_size 1.524 2.54)
     (pad_drill 0)
     (pad_to_mask_clearance 0)
@@
     )
     (pad 2 smd rect (at -2.54 0 180) (size 1.524 2.54)
-      (layers B.Cu F.Paste F.Mask)
+      (layers *.Mask B.Cu F.Paste)
       (net 2 +5V)
     )
     (pad 4 smd rect (at 0 0 180) (size 1.524 2.54)
-      (layers B.Cu F.Paste F.Mask)
+      (layers *.Mask B.Cu F.Paste)
       (net 5 N-0000013)
     )
     (pad 6 smd rect (at 2.54 0 180) (size 1.524 2.54)
-      (layers B.Cu F.Paste F.Mask)
-      (net 3 GND)
-    )
+      (layers *.Mask B.Cu F.Paste)
+      (net 3 GND)
+    )
+  )
+  (gr_text "NOTE:\nCan shorten the USB part a tad.  I.e. 1/6th the length of the item." (at 68.58 56.4642) (layer Dwgs.User)
+    (effects (font (size 0.762 0.762) (thickness 0.1524)))
   )
   (gr_text MISO (at 56.8 54.8 90) (layer F.SilkS)
