File: usb_minecraft/hw/usb_minecraft.sch (KiCad schematic (older format))
At the start: 9 parts, among them J1 AVRISP6, P1 USB, U1 ATMEGAXU2, U2 10p, U3 1u, U4 33, X1 16MHz

Commit message: Yay updates
Other:
- note added: "WARNING:\nSee PCB doc for notes.\n\nChanges:\n(1) Skip 33 ohm network\n(2) Use 2 capacitors instead of 4xnetwork."
Changed lines of the file:
@@
 LIBS:rs485-isl3170
 LIBS:um5k1ntr
-LIBS:ATMegaBB-cache
+LIBS:usb_minecraft-cache
 EELAYER 27 0
 EELAYER END
@@
 Sheet 1 1
 Title ""
-Date "22 oct 2014"
+Date "27 nov 2014"
 Rev ""
 Comp ""
@@
 	4800 5350 4800 5800
 Connection ~ 6650 6250
+Text Notes 1650 5050 0    60   ~ 0
+WARNING:\nSee PCB doc for notes.\n\nChanges:\n(1) Skip 33 ohm network\n(2) Use 2 capacitors instead of 4xnetwork.
 $EndSCHEMATC
